Commit message: semubot_description

File: install/semubot_description/share/semubot_description/urdf/head.urdf.xacro (robot description, xacro)
@@ -1 +1,82 @@
-/home/mykyta-nesterenko/Nesterenko-thesis-2026-ROS-stack/src/semubot_description/urdf/head.urdf.xacro
+<?xml version="1.0"?>
+<robot xmlns:xacro="http://www.ros.org/wiki/xacro">
+  <xacro:macro name="head_macro" params="parent xyz rpy">
+    <!-- Head Base -->
+    <link name="head_base">
+      <visual>
+        <geometry>
+          <mesh filename="package://semubot_description/meshes/head_base.stl" scale="1 1 1"/>
+        </geometry>
+        <material name="white"/>
+      </visual>
+      <collision>
+        <origin xyz="0 0 0" rpy="0 0 0"/>
+        <geometry>
+          <cylinder radius="0.06" length="0.1"/>
+        </geometry>
+      </collision>
+      <inertial>
+        <origin xyz="0 0 0" rpy="0 0 0"/>
+        <mass value="0.4"/>
+        <inertia ixx="0.01" ixy="0.0" ixz="0.0" iyy="0.01" iyz="0.0" izz="0.01"/>
+      </inertial>
+    </link>
+    <joint name="head_joint" type="revolute">
+      <parent link="${parent}"/>
+      <child link="head_base"/>
+      <origin xyz="${xyz}" rpy="${rpy}"/>
+      <axis xyz="0 1 0"/>
+      <limit lower="-1.57" upper="1.57" effort="10" velocity="1.0"/>
+    </joint>
+    <!-- Head Scalp -->
+    <link name="head_scalp">
+      <visual>
+        <geometry>
+          <mesh filename="package://semubot_description/meshes/head_scalp.stl" scale="1 1 1"/>
+        </geometry>
+        <material name="cyan"/>
+      </visual>
+      <collision>
+        <origin xyz="0 0 0.12" rpy="0 0 0"/>
+        <geometry>
+          <sphere radius="0.12"/>
+        </geometry>
+      </collision>
+      <inertial>
+        <origin xyz="0 0 0" rpy="0 0 0"/>
+        <mass value="0.2"/>
+        <inertia ixx="0.005" ixy="0.0" ixz="0.0" iyy="0.005" iyz="0.0" izz="0.005"/>
+      </inertial>
+    </link>
+    <joint name="head_scalp_joint" type="fixed">
+      <parent link="head_base"/>
+      <child link="head_scalp"/>
+      <origin xyz="0 0 0" rpy="0 0 0"/>
+    </joint>
+    <!-- Head Screen -->
+    <link name="head_screen">
+      <visual>
+        <geometry>
+          <mesh filename="package://semubot_description/meshes/head_screen.stl" scale="1 1 1"/>
+        </geometry>
+        <material name="black"/>
+      </visual>
+      <collision>
+        <origin xyz="0 0 0" rpy="0 0 0"/>
+        <geometry>
+          <box size="0.1 0.01 0.08"/>
+        </geometry>
+      </collision>
+      <inertial>
+        <origin xyz="0 0 0" rpy="0 0 0"/>
+        <mass value="0.2"/>
+        <inertia ixx="0.005" ixy="0.0" ixz="0.0" iyy="0.005" iyz="0.0" izz="0.005"/>
+      </inertial>
+    </link>
+    <joint name="head_screen_joint" type="fixed">
+      <parent link="head_base"/>
+      <child link="head_screen"/>
+      <origin xyz="0 0 0" rpy="0 0 0"/>
+    </joint>
+  </xacro:macro>
+</robot>

File: install/semubot_description/share/semubot_description/urdf/semubot.urdf.xacro (robot description, xacro)
@@ -1 +1,199 @@
-/home/mykyta-nesterenko/Nesterenko-thesis-2026-ROS-stack/src/semubot_description/urdf/semubot.urdf.xacro
+<?xml version="1.0"?>
+<robot xmlns:xacro="http://www.ros.org/wiki/xacro" name="semubot">
+  <xacro:include filename="$(find semubot_description)/urdf/head.urdf.xacro"/>
+  <material name="white">
+    <color rgba="1 1 1 1"/>
+  </material>
+  <material name="cyan">
+    <color rgba="0 1 1 1"/>
+  </material>
+  <material name="black">
+    <color rgba="0 0 0 1"/>
+  </material>
+  <!-- Base Link -->
+  <link name="base_link">
+    <visual>
+      <origin xyz="0 0 0.04" rpy="0 0 0"/>
+      <geometry>
+        <mesh filename="package://semubot_description/meshes/movement_frame.stl" scale="1 1 1"/>
+      </geometry>
+      <material name="white"/>
+    </visual>
+    <collision>
+      <origin xyz="0 0 0.2" rpy="0 0 0"/>
+      <geometry>
+        <cylinder radius="0.28" length="0.3"/>
+      </geometry>
+    </collision>
+    <inertial>
+      <origin xyz="0 0 0.02" rpy="0 0 0"/>
+      <mass value="5.0"/>
+      <inertia ixx="0.1" ixy="0.0" ixz="0.0" iyy="0.1" iyz="0.0" izz="0.1"/>
+    </inertial>
+  </link>
+  <!-- Macro for Omni-ball -->
+  <xacro:macro name="omni_ball_macro" params="name xyz rpy scale mass ixx iyy izz">
+    <link name="${name}">
+      <visual>
+        <origin xyz="0 0 0" rpy="0 0 0"/>
+        <geometry>
+          <mesh filename="package://semubot_description/meshes/omni_ball.stl" scale="${scale} ${scale} ${scale}"/>
+        </geometry>
+        <material name="white"/>
+      </visual>
+      <collision>
+        <origin xyz="0 0 0" rpy="0 0 0"/>
+        <geometry>
+          <sphere radius="0.06"/>
+        </geometry>
+      </collision>
+      <inertial>
+        <origin xyz="0 0 0" rpy="0 0 0"/>
+        <mass value="${mass}"/>
+        <inertia ixx="${ixx}" ixy="0.0" ixz="0.0" iyy="${iyy}" iyz="0.0" izz="${izz}"/>
+      </inertial>
+    </link>
+  </xacro:macro>
+  <!-- Omni-balls -->
+  <xacro:omni_ball_macro name="omni_ball_1" xyz="0 0 0" rpy="0 0 0" scale="1" mass="0.1" ixx="0.001" iyy="0.001" izz="0.001"/>
+  <xacro:omni_ball_macro name="omni_ball_2" xyz="0 0 0" rpy="0 0 0" scale="1" mass="0.1" ixx="0.001" iyy="0.001" izz="0.001"/>
+  <xacro:omni_ball_macro name="omni_ball_3" xyz="0 0 0" rpy="0 0 0" scale="1" mass="0.1" ixx="0.001" iyy="0.001" izz="0.001"/>
+  <!-- Joints for Omni-balls -->
+  <joint name="omni_ball_1_joint" type="continuous">
+    <parent link="base_link"/>
+    <child link="omni_ball_1"/>
+    <origin xyz="0.16 0.265 0.06" rpy="0 0 ${2*pi/3}"/>
+    <axis xyz="1 0 0"/>
+    <limit effort="50" velocity="1.0"/>
+  </joint>
+  <joint name="omni_ball_2_joint" type="continuous">
+    <parent link="base_link"/>
+    <child link="omni_ball_2"/>
+    <origin xyz="0.16 -0.265 0.06" rpy="0 0 ${-2*pi/3}"/>
+    <axis xyz="1 0 0"/>
+    <limit effort="50" velocity="1.0"/>
+  </joint>
+  <joint name="omni_ball_3_joint" type="continuous">
+    <parent link="base_link"/>
+    <child link="omni_ball_3"/>
+    <origin xyz="-0.3 0 0.06" rpy="0 0 0"/>
+    <axis xyz="1 0 0"/>
+    <limit effort="50" velocity="1.0"/>
+  </joint>
+  <!-- Main Body -->
+  <link name="main_body">
+    <visual>
+      <geometry>
+        <mesh filename="package://semubot_description/meshes/body.stl" scale="1 1 1"/>
+      </geometry>
+      <material name="white"/>
+    </visual>
+    <collision>
+      <origin xyz="0.01 0 0.4" rpy="0 0 0"/>
+      <geometry>
+        <cylinder radius="0.17" length="0.5"/>
+      </geometry>
+    </collision>
+    <inertial>
+      <origin xyz="0 0 0.05" rpy="0 0 0"/>
+      <mass value="3.0"/>
+      <inertia ixx="0.05" ixy="0.0" ixz="0.0" iyy="0.05" iyz="0.0" izz="0.05"/>
+    </inertial>
+  </link>
+  <joint name="body_joint" type="fixed">
+    <parent link="base_link"/>
+    <child link="main_body"/>
+    <origin xyz="0 0 0.045" rpy="0 0 0"/>
+  </joint>
+  <!-- Left Arm -->
+  <link name="left_arm">
+    <visual>
+      <geometry>
+        <mesh filename="package://semubot_description/meshes/left_hand.stl" scale="1 1 1"/>
+      </geometry>
+      <material name="white"/>
+    </visual>
+    <collision>
+      <origin xyz="0 0.05 -0.1" rpy="0 0 0"/>
+      <geometry>
+        <cylinder radius="0.03" length="0.3"/>
+      </geometry>
+    </collision>
+    <inertial>
+      <origin xyz="0 0 0" rpy="0 0 0"/>
+      <mass value="0.5"/>
+      <inertia ixx="0.01" ixy="0.0" ixz="0.0" iyy="0.01" iyz="0.0" izz="0.01"/>
+    </inertial>
+  </link>
+  <joint name="left_arm_joint" type="revolute">
+    <parent link="main_body"/>
+    <child link="left_arm"/>
+    <origin xyz="0 0.175 0.555" rpy="0 0 0"/>
+    <axis xyz="0 1 0"/>
+    <limit lower="-1.57" upper="1.57" effort="10" velocity="1.0"/>
+  </joint>
+  <!-- Right Arm -->
+  <link name="right_arm">
+    <visual>
+      <geometry>
+        <mesh filename="package://semubot_description/meshes/right_hand.stl" scale="1 1 1"/>
+      </geometry>
+      <material name="white"/>
+    </visual>
+    <collision>
+      <origin xyz="0 -0.05 -0.1" rpy="0 0 0"/>
+      <geometry>
+        <cylinder radius="0.03" length="0.3"/>
+      </geometry>
+    </collision>
+    <inertial>
+      <origin xyz="0 0 0" rpy="0 0 0"/>
+      <mass value="0.5"/>
+      <inertia ixx="0.01" ixy="0.0" ixz="0.0" iyy="0.01" iyz="0.0" izz="0.01"/>
+    </inertial>
+  </link>
+  <joint name="right_arm_joint" type="revolute">
+    <parent link="main_body"/>
+    <child link="right_arm"/>
+    <origin xyz="0 -0.175 0.555" rpy="0 0 0"/>
+    <axis xyz="0 1 0"/>
+    <limit lower="-1.57" upper="1.57" effort="10" velocity="1.0"/>
+  </joint>
+  <!-- Head -->
+  <xacro:head_macro parent="main_body" xyz="0 0 0.705" rpy="0 0 0"/>
+  <!-- ros2_control Hardware Interface -->
+<ros2_control name="SemubotHardwareSystem" type="system">
+  <hardware>
+    <plugin>semubot_hardware_interface/SemubotHardwareInterface</plugin>
+    <param name="wheel_radius">0.06</param>
+    <param name="base_radius">0.305</param>
+  </hardware>
+  <joint name="omni_ball_1_joint">
+    <command_interface name="velocity">
+      <param name="min">-10.0</param>
+      <param name="max">10.0</param>
+    </command_interface>
+    <state_interface name="position"/>
+    <state_interface name="velocity"/>
+    <state_interface name="effort"/>
+  </joint>
+  <joint name="omni_ball_2_joint">
+    <command_interface name="velocity">
+      <param name="min">-10.0</param>
+      <param name="max">10.0</param>
+    </command_interface>
+    <state_interface name="position"/>
+    <state_interface name="velocity"/>
+    <state_interface name="effort"/>
+  </joint>
+  <joint name="omni_ball_3_joint">
+    <command_interface name="velocity">
+      <param name="min">-10.0</param>
+      <param name="max">10.0</param>
+    </command_interface>
+    <state_interface name="position"/>
+    <state_interface name="velocity"/>
+    <state_interface name="effort"/>
+  </joint>
+</ros2_control>
+</robot>
